File: minivan-clone.kicad_pcb (KiCad board)
At the start: 2 copper layers, 117 parts, among them CON101 HRO-TYPE-C-31-M-12, CON102 CONN_3X2, K101 KEYSW, K102 KEYSW, K103 KEYSW, K104 KEYSW, K105 KEYSW, K106 KEYSW, K107 KEYSW, K108 KEYSW, K110 KEYSW, K111 KEYSW, K112 KEYSW, K113 KEYSW, K114 KEYSW, K115 KEYSW, K116 KEYSW, K117 KEYSW, K118 KEYSW, K119 KEYSW, K120 KEYSW, K121 KEYSW, K122 KEYSW, K123 KEYSW, K124 KEYSW, K125 KEYSW, K126 KEYSW, K127 KEYSW, K128 KEYSW, K129 KEYSW, K130 KEYSW, K131 KEYSW, K132 KEYSW, K133 KEYSW, K134 KEYSW, K135 KEYSW, K136 KEYSW, K137 KEYSW, K138 KEYSW, K139 KEYSW, K140 KEYSW, K141 KEYSW, K142 KEYSW, K143 KEYSW, K144 KEYSW, K145 KEYSW, K146 KEYSW, K147 KEYSW, K148 KEYSW, SW101 SW_PUSH, U101 ATMEGA32U2, X101 XTAL_GND

Commit message: started layout
started layout
Parts:
- K113: footprint keebs:Mx_Alps_100 -> keebs:Mx_Alps_175
- K115: footprint keebs:Mx_Alps_100 -> keebs:Mx_Alps_125
- K126: footprint keebs:Mx_Alps_100 -> keebs:Mx_Alps_150
- moved K140 362.6 mm to (189.0, 216.0)
- moved K130 358.9 mm to (228.4, 193.3)
- moved K114 290.2 mm to (459.0, 104.0)
- moved K144 269.6 mm to (265.0, 216.0)
- moved K135 251.3 mm to (318.0, 194.0)
- moved K101 222.8 mm to (130.0, 138.0)
- moved K102 211.6 mm to (149.1, 138.0)
- moved K115 207.3 mm to (132.4, 157.1)
- moved K104 204.2 mm to (187.2, 138.0)
- moved K103 201.6 mm to (168.1, 138.0)
- moved K105 187.3 mm to (206.2, 138.0)
- moved K108 184.6 mm to (263.4, 138.0)
- moved K124 183.2 mm to (310.4, 157.1)
- moved K148 183.0 mm to (341.0, 214.0)
- moved K116 180.4 mm to (153.8, 157.1)
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
Commit message: fixed row 2
Parts:
- K113: footprint keebs:Mx_Alps_175 -> keebs:Mx_Alps_100
- K126: footprint keebs:Mx_Alps_150 -> keebs:Mx_Alps_175
- K127: footprint keebs:Mx_Alps_100 -> keebs:Mx_Alps_175
- moved K138 219.0 mm to (363.2, 176.5)
- moved K137 214.9 mm to (339.1, 177.8)
- moved K114 106.0 mm to (358.6, 138.0)
- moved K127 48.2 mm to (125.2, 176.1)
- moved K128 27.1 mm to (166.4, 179.1)
- moved K134 26.4 mm to (278.3, 178.8)
- moved K129 26.4 mm to (187.4, 178.8)
- moved K130 26.4 mm to (206.8, 178.0)
- moved K131 26.4 mm to (223.4, 177.8)
- moved K132 26.4 mm to (243.4, 178.8)
- moved K133 26.4 mm to (260.4, 178.8)
- moved K135 26.4 mm to (296.4, 178.8)
- moved K136 26.4 mm to (315.4, 177.8)
- moved K113 8.33 mm to (339.6, 138.0)
- moved K125 4.76 mm to (325.3, 157.1)
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
Commit message: added -bak and -rescue* to gitignore
Parts:
- K138, K142, K145: footprint keebs:Mx_Alps_100 -> keebs:Mx_Alps_125
- K143, K144: footprint keebs:Mx_Alps_100 -> keebs:Mx_Alps_225
- moved K140 45.1 mm to (149.1, 195.2)
- moved K141 45.0 mm to (168.1, 195.2)
- moved K139 44.3 mm to (130.0, 195.2)
- moved K142 43.4 mm to (189.5, 195.2)
- moved K147 41.6 mm to (358.6, 195.2)
- moved K143 31.1 mm to (222.9, 195.2)
- moved K146 27.1 mm to (320.5, 195.2)
- moved K145 25.5 mm to (299.1, 195.2)
- moved K144 20.9 mm to (265.7, 195.2)
- moved K148 18.9 mm to (339.6, 195.2)
- moved K127 11.9 mm to (137.1, 176.1)
- moved K138 7.01 mm to (356.2, 176.1)
- moved K130 5.71 mm to (201.4, 176.1)
- moved K129 5.68 mm to (182.4, 176.1)
- moved K132 4.70 mm to (239.5, 176.1)
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
Commit message: placed all connected diods
Parts:
- added >NAME: >VALUE, keebs:Mx_Alps_200, F.Cu at (349.1, 138.0)
- moved D113 277.0 mm to (367.3, 141.4), turned to 90 degrees
- moved D137 264.2 mm to (364.7, 179.3), turned to 90 degrees
- moved D146 247.3 mm to (367.3, 198.1), turned to 90 degrees
- moved D125 246.4 mm to (360.2, 160.5), turned to 90 degrees
- moved D110 245.2 mm to (309.9, 141.2), turned to 90 degrees
- moved D136 244.6 mm to (343.4, 179.3), turned to 90 degrees
- moved PTC101 237.3 mm to (143.5, 143.5)
- moved C106 233.1 mm to (137.2, 139.7)
- moved D108 225.1 mm to (271.8, 141.2), turned to 90 degrees
- moved D134 224.0 mm to (305.3, 179.3), turned to 90 degrees
- moved D148 220.2 mm to (136.8, 145.3)
- moved D101 218.9 mm to (121.9, 143.3), turned to 90 degrees
- moved D109 216.5 mm to (291.1, 141.2), turned to 90 degrees
- moved X101 213.8 mm to (238.4, 181.4)
- moved D107 212.4 mm to (253.0, 141.2), turned to 90 degrees
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
Commit message: added missing connections for diods, diods on pcb
Parts:
- moved D102 144.7 mm to (157.5, 141.2), turned to 90 degrees
- moved D103 139.8 mm to (176.3, 141.2), turned to 90 degrees
- moved D116 137.9 mm to (181.4, 160.0), turned to 90 degrees
- moved D111 113.5 mm to (329.2, 141.2), turned to 90 degrees
- moved D112 112.1 mm to (348.0, 142.2), turned to 90 degrees
- moved D135 101.6 mm to (324.1, 179.3), turned to 90 degrees
- moved D124 92.5 mm to (333.8, 160.0), turned to 90 degrees
- moved D122 78.2 mm to (295.7, 160.0), turned to 90 degrees
- moved D123 72.8 mm to (315.0, 160.0), turned to 90 degrees
- moved R106 44.8 mm to (215.9, 322.1)
- moved D113 0.85 mm to (367.3, 142.2)
Connections:
- K102 pad 2: Net-(K102-Pad2) -> Net-(D102-Pad2)
- K103 pad 2: Net-(K103-Pad2) -> Net-(D103-Pad2)
- K112 pad 2: Net-(K112-Pad2) -> Net-(D111-Pad2)
- K113 pad 2: Net-(K113-Pad2) -> Net-(D112-Pad2)
- K117 pad 2: Net-(K117-Pad2) -> Net-(D116-Pad2)
- K123 pad 2: Net-(K123-Pad2) -> Net-(D122-Pad2)
- K124 pad 2: Net-(K124-Pad2) -> Net-(D123-Pad2)
- K125 pad 2: Net-(K125-Pad2) -> Net-(D124-Pad2)
- K136 pad 2: Net-(K136-Pad2) -> Net-(D135-Pad2)

Commit message: removed ICSP, fixed gnd and 5v
Parts:
- added D202: PRTR5V0U2X, Package_TO_SOT_SMD:SOT-143, F.Cu at (125.5, 294.1)
- moved C106 2.96 mm to (134.6, 141.2)
- moved D125 0.51 mm to (360.2, 160.0)
Connections:
- C101 pad 2: +5V -> GND
- C102 pad 2: +5V -> GND
- C103 pad 2: +5V -> GND
- C104 pad 2: +5V -> GND
- C105 pad 2: +5V -> GND
- C106 pad 2: +5V -> GND
- C107 pad 2: +5V -> GND
- C108 pad 2: +5V -> GND
- C109 pad 2: +5V -> GND
- C110 pad 1: +5V -> GND
- CON101 pad 1: +5V -> GND
- CON101 pad 12: +5V -> GND
- CON101 pad 13: +5V -> GND
- CON102 pad 2: +5V -> Net-(CON102-Pad2)
- D148 pad 1: +5V -> Net-(D148-Pad1)
- D148 pad 4: +5V -> Net-(D148-Pad4)
- R102 pad 2: +5V -> GND
- R105 pad 2: +5V -> GND
- R106 pad 2: +5V -> GND
- SW101 pad 2: +5V -> GND
- U101 pad 28: +5V -> GND
- U101 pad 3: +5V -> GND
- X101 pad 3: +5V -> GND

Commit message: placed processor and usb components
Parts:
- removed CON102: CONN_3X2, keyboard_parts:AVR_ICSP_3x2
- removed D148: PRTR5V0U2X, Package_TO_SOT_SMD:SOT-143
- moved R105 228.8 mm to (142.7, 142.7), turned to 270 degrees
- moved R106 196.5 mm to (135.6, 142.7), turned to 270 degrees
- moved C102 195.0 mm to (237.2, 194.1), turned to 180 degrees
- moved C101 194.7 mm to (237.2, 196.1), turned to 180 degrees
- moved C110 187.0 mm to (233.7, 192.0), turned to 90 degrees
- moved C109 181.5 mm to (245.9, 206.2)
- moved C104 169.7 mm to (229.4, 216.7)
- moved C105 169.7 mm to (214.8, 224.5)
- moved SW101 169.7 mm to (238.8, 223.5)
- moved R102 169.7 mm to (239.1, 214.8)
- moved C103 168.8 mm to (243.3, 201.7), turned to 270 degrees
- moved R101 164.1 mm to (254.5, 221.5)
- moved D202 154.5 mm to (139.1, 140.2), turned to 180 degrees
- moved R104 14.4 mm to (230.4, 208.5)
- moved C108 13.5 mm to (234.2, 198.1), turned to 90 degrees
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
Commit message: Started routing
Started routing
Parts:
- removed C104: 0,1uF, keyboard_parts:C_1608_rev2
- C110: footprint keyboard_parts:C_3216_rev2 -> keyboard_parts:C_1608_rev2
- moved SW101 42.9 mm to (239.5, 180.6), turned to 180 degrees
- moved C105 40.9 mm to (228.6, 185.9), turned to 90 degrees
- moved R101 39.1 mm to (239.5, 185.4), turned to 90 degrees
- moved R102 25.8 mm to (252.5, 192.8)
- moved C109 21.3 mm to (241.3, 185.4), turned to 90 degrees
- moved D146 19.1 mm to (348.2, 198.1)
- moved K147 19.1 mm to (339.6, 195.2)
- moved K148 19.1 mm to (358.6, 195.2)
- moved D147 17.5 mm to (365.5, 198.1)
- moved X101 17.1 mm to (242.8, 201.9)
- moved D137 17.0 mm to (347.7, 179.3)
- moved R104 15.7 mm to (232.7, 193.0)
- moved D113 15.0 mm to (352.3, 142.2)
- moved C108 12.7 mm to (246.4, 201.7), turned to 270 degrees
- moved R103 9.49 mm to (232.7, 195.1)
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Connections:
- >NAME pad 2: Net-(K113-Pad2) -> Net-(D112-Pad2)
- CON101 pad 5: Net-(CON101-Pad5) -> /pre_D+
- CON101 pad 6: Net-(CON101-Pad6) -> /pre_D-
- CON101 pad 7: Net-(CON101-Pad5) -> /pre_D+
- CON101 pad 8: Net-(CON101-Pad6) -> /pre_D-
- D101 pad 1: /PD0 -> /PB3
- D102 pad 1: /PD0 -> /PB3
- D103 pad 1: /PD0 -> /PB3
- D104 pad 1: /PD0 -> /PB3
- D105 pad 1: /PD0 -> /PB3
- D106 pad 1: /PD0 -> /PB3
- D107 pad 1: /PD0 -> /PB3
- D108 pad 1: /PD0 -> /PB3
- D109 pad 1: /PD0 -> /PB3
- D110 pad 1: /PD0 -> /PB3
- D111 pad 1: /PD0 -> /PB3
- D112 pad 1: /PD0 -> /PB3
- D113 pad 1: /PD0 -> /PB3
- D114 pad 1: /PD1 -> /PB1
- D115 pad 1: /PD1 -> /PB1
- D116 pad 1: /PD1 -> /PB1
- D117 pad 1: /PD1 -> /PB1
- D118 pad 1: /PD1 -> /PB1
- D119 pad 1: /PD1 -> /PB1
- D120 pad 1: /PD1 -> /PB1
- D121 pad 1: /PD1 -> /PB1
- D122 pad 1: /PD1 -> /PB1
- D123 pad 1: /PD1 -> /PB1
- D124 pad 1: /PD1 -> /PB1
- D125 pad 1: /PD1 -> /PB1
- D126 pad 1: /PD2 -> /PB2
- D127 pad 1: /PD2 -> /PB2
- D128 pad 1: /PD2 -> /PB2
- D129 pad 1: /PD2 -> /PB2
- D130 pad 1: /PD2 -> /PB2
- D131 pad 1: /PD2 -> /PB2
- D132 pad 1: /PD2 -> /PB2
- D133 pad 1: /PD2 -> /PB2
- D134 pad 1: /PD2 -> /PB2
- D135 pad 1: /PD2 -> /PB2
- D136 pad 1: /PD2 -> /PB2
- D137 pad 1: /PD2 -> /PB2
- D138 pad 1: /PD4 -> /PC2
- D139 pad 1: /PD4 -> /PC2
- D140 pad 1: /PD4 -> /PC2
- D141 pad 1: /PD4 -> /PC2
- D142 pad 1: /PD4 -> /PC2
- D143 pad 1: /PD4 -> /PC2
- D144 pad 1: /PD4 -> /PC2
- D145 pad 1: /PD4 -> /PC2
- D146 pad 1: /PD4 -> /PC2
- D147 pad 1: /PD4 -> /PC2
- D202 pad 2: /D- -> /pre_D+
- D202 pad 3: /D+ -> /pre_D-
- K107 pad 1: /MISO -> /PD0
- K108 pad 1: /MOSI -> /PD2
- K110 pad 1: /PB1 -> /PD3
- K111 pad 1: /PB0 -> /PD4
- K112 pad 1: /PD6 -> /PD5
- K113 pad 1: /PD5 -> /PB0
- K114 pad 1: /PC2 -> /PD6
- K121 pad 1: /MISO -> /PD0
- K122 pad 1: /MOSI -> /PD2
- K123 pad 1: /PB1 -> /PD3
- K124 pad 1: /PB0 -> /PD4
- K125 pad 1: /PD6 -> /PD5
- K126 pad 1: /PD5 -> /PB0
- K133 pad 1: /MISO -> /PD0
- K134 pad 1: /MOSI -> /PD2
- K135 pad 1: /PB1 -> /PD3
- K136 pad 1: /PB0 -> /PD4
- K137 pad 1: /PD6 -> /PD5
- K138 pad 1: /PD5 -> /PB0
- K144 pad 1: /MISO -> /PD0
- K145 pad 1: /MOSI -> /PD2
- K146 pad 1: /PB1 -> /PD3
- K147 pad 1: /PB0 -> /PD4
- K148 pad 1: /PD6 -> /PD5
- R103 pad 1: Net-(CON101-Pad6) -> /pre_D-
- R104 pad 1: Net-(CON101-Pad5) -> /pre_D+
- U101 pad 16: /MOSI -> /PB2
- U101 pad 17: /MISO -> /PB3
- U101 pad 29: /DP -> /D+
- U101 pad 30: /DN -> /D-
Routing:
- net /PD5: track 0.00 -> 251.1 mm
- net /PC2: track 0.00 -> 245.6 mm, vias 0 -> 2
- net /PB3: track 0.00 -> 227.7 mm, vias 0 -> 2
- net /PB2: track 0.00 -> 221.4 mm, vias 0 -> 2
- net /PB1: track 0.00 -> 220.9 mm, vias 0 -> 2
- net +5V: track 0.00 -> 178.9 mm, vias 0 -> 2
- net /PD4: track 0.00 -> 173.3 mm
- net /PD6: track 0.00 -> 164.4 mm
- net /PD3: track 0.00 -> 153.6 mm
- net /pre_D-: track 0.00 -> 135.6 mm
- net /pre_D+: track 0.00 -> 134.7 mm
- net /PD2: track 0.00 -> 129.8 mm
- net /PB0: track 0.00 -> 116.8 mm
- net /PD0: track 0.00 -> 116.6 mm
- net /PB6: track 0.00 -> 91.2 mm
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