File: matrix.sch (KiCad schematic (older format))
At the start: 0 parts

Commit message: done work on mcu and started on matrix
done work on mcu and started on matrix
Parts:
- added D101, D102, D103, D104, D105, D106, D107, D108, D109, D110, D111, D112, D113, D114, D115, D116, D117, D118, D119, D120, D121, D122, D123, D124, D125, D126, D127, D128, D129, D130, D131, D132, D133, D134, D135, D136, D137, D138, D139, D140, D141, D142, D143, D144, D145, D146, D147: D, symbol keyboard_parts:D
- added K101, K102, K103, K104, K105, K106, K107, K108, K110, K111, K112, K113, K114, K115, K116, K117, K118, K119, K120, K121, K122, K123, K124, K125, K126, K127, K128, K129, K130, K131, K132, K133, K134, K135, K136, K137, K138, K139, K140, K141, K142, K143, K144, K145, K146, K147, K148: KEYSW, symbol keyboard_parts:KEYSW
Connections:
- new net: D101.2, K101.2
- new net: D104.2, K104.2
- new net: D105.2, K105.2
- new net: D106.2, K106.2
- new net: D107.2, K107.2
- new net: D108.2, K108.2
- new net: D109.2, K110.2
- new net: D110.2, K111.2
- new net: D113.2, K114.2
- new net: D117.2, K118.2
- new net: D118.2, K119.2
- new net: D119.2, K120.2
- new net: D114.2, K115.2
- new net: D115.2, K116.2
- new net: D120.2, K121.2
- new net: D121.2, K122.2
- new net: D125.2, K126.2
- new net: D129.2, K130.2
- new net: D130.2, K131.2
- new net: D131.2, K132.2
- new net: D126.2, K127.2
- new net: D127.2, K128.2
- new net: D128.2, K129.2
- new net: D132.2, K133.2
- new net: D133.2, K134.2
- new net: D134.2, K135.2
- new net: D136.2, K137.2
- new net: D137.2, K138.2
- new net: D141.2, K142.2
- new net: D142.2, K143.2
- new net: D143.2, K144.2
- new net: D138.2, K139.2
- new net: D139.2, K140.2
- new net: D140.2, K141.2
- new net: D144.2, K145.2
- new net: D145.2, K146.2
- new net: D146.2, K147.2
- new net: D147.2, K148.2
- new net COL1: K101.1, K115.1, K127.1
- new net COL10: K111.1, K124.1, K136.1, K147.1
- new net COL11: K112.1, K125.1, K137.1, K148.1
- new net COL12: K113.1, K126.1, K138.1
- new net COL13: K114.1
- new net COL2: K102.1, K116.1, K128.1, K139.1
- new net COL3: K103.1, K117.1, K129.1, K140.1
- new net COL4: K104.1, K118.1, K130.1, K141.1
- new net COL5: K105.1, K119.1, K131.1, K142.1
- new net COL6: K106.1, K120.1, K132.1, K143.1
- new net COL7: K107.1, K121.1, K133.1, K144.1
- new net COL8: K108.1, K122.1, K134.1, K145.1
- new net COL9: K110.1, K123.1, K135.1, K146.1
- new net ROW1: D101.1, D102.1, D103.1, D104.1, D105.1, D106.1, D107.1, D108.1, D109.1, D110.1, D111.1, D112.1, D113.1
- new net ROW2: D114.1, D115.1, D116.1, D117.1, D118.1, D119.1, D120.1, D121.1, D122.1, D123.1, D124.1, D125.1
- new net ROW3: D126.1, D127.1, D128.1, D129.1, D130.1, D131.1, D132.1, D133.1, D134.1, D135.1, D136.1, D137.1
- new net ROW4: D138.1, D139.1, D140.1, D141.1, D142.1, D143.1, D144.1, D145.1, D146.1, D147.1

Commit message: started doing layout
started doing layout
Parts:
- D101, D102, D103, D104, D105, D106, D107, D108, D109, D110, D111, D112, D113, D114, D115, D116, D117, D118, D119, D120, D121, D122, D123, D124, D125, D126, D127, D128, D129, D130, D131, D132, D133, D134, D135, D136, D137, D138, D139, D140, D141, D142, D143, D144, D145, D146, D147: footprint (none) -> keyboard_parts:D_SC79
- K101, K102, K103, K104, K105, K106, K107, K108, K110, K111, K112, K113, K114, K115, K116, K117, K118, K119, K120, K121, K122, K123, K124, K125, K126, K127, K128, K129, K130, K131, K132, K133, K134, K135, K136, K137, K138, K139, K140, K141, K142, K143, K144, K145, K146, K147, K148: footprint (none) -> keebs:Mx_Alps_100

Commit message: added missing connections for diods, diods on pcb
Connections:
- net at D102.2: now also K102.2
- net at D103.2: now also K103.2
- net at K112.2: now also D111.2
- net at K113.2: now also D112.2
- net at K117.2: now also D116.2
- net at K123.2: now also D122.2
- net at K124.2: now also D123.2
- net at K125.2: now also D124.2
- net at K136.2: now also D135.2
Changed lines of the file:
@@
 	1    0    0    -1
 $EndComp
+Wire Wire Line
+	4400 4150 4400 4300
+Wire Wire Line
+	5200 4150 5200 4300
+Wire Wire Line
+	11550 4150 11550 4300
+Wire Wire Line
+	12350 4300 12350 4150
+Wire Wire Line
+	10650 5100 10650 5250
+Wire Wire Line
+	11450 5100 11450 5250
+Wire Wire Line
+	9850 5100 9850 5250
+Wire Wire Line
+	5150 5100 5150 5250
+Wire Wire Line
+	10600 5950 10600 6100
 $EndSCHEMATC

Commit message: Mirroring layout
Parts:
- renumbered K114 to K101, K113 to K102, K112 to K103, K111 to K104, K110 to K105, K108 to K106, K106 to K108, K105 to K109, K104 to K110, K103 to K111, K102 to K112, K101 to K113, K126 to K114, K125 to K115, K124 to K116, K123 to K118, K122 to K119, K121 to K120, K120 to K121, K119 to K122, K118 to K123, K117 to K124, K116 to K125, K115 to K126, K138 to K127, K137 to K128, K136 to K129, K135 to K130, K134 to K131, K133 to K132, K132 to K133, K131 to K134, K130 to K135, K129 to K136, K128 to K137, K127 to K138, K148 to K139, K147 to K140, K146 to K141, K145 to K142, K144 to K143, K143 to K144, K142 to K145, K141 to K146, K140 to K147, K139 to K148
