File: plate.kicad_pcb (KiCad board)
At the start: 2 copper layers, 247.4 x 75.9 mm, 47 parts, among them K101 KEYSW, K102 KEYSW, K103 KEYSW, K104 KEYSW, K105 KEYSW, K106 KEYSW, K107 KEYSW, K108 KEYSW, K109 KEYSW, K110 KEYSW, K111 KEYSW, K112 KEYSW, K113 KEYSW, K114 KEYSW, K115 KEYSW, K116 KEYSW, K118 KEYSW, K119 KEYSW, K120 KEYSW, K121 KEYSW, K122 KEYSW, K123 KEYSW, K124 KEYSW, K125 KEYSW, K126 KEYSW, K127 KEYSW, K128 KEYSW, K129 KEYSW, K130 KEYSW, K131 KEYSW, K132 KEYSW, K133 KEYSW, K134 KEYSW, K135 KEYSW, K136 KEYSW, K137 KEYSW, K138 KEYSW, K139 KEYSW, K140 KEYSW, K141 KEYSW, K142 KEYSW, K143 KEYSW, K144 KEYSW, K145 KEYSW, K146 KEYSW, K147 KEYSW, K148 KEYSW

Commit message: plate has increased size with 6mm
Parts:
- added HOLE_M3: VAL**, keyboard_parts:HOLE_M3, F.Cu at (245.9, 208.4)
- added HOLE_M3: VAL**, keyboard_parts:HOLE_M3, F.Cu at (245.9, 125.8)
- added HOLE_M3: VAL**, keyboard_parts:HOLE_M3, F.Cu at (370.3, 127.1)
- added HOLE_M3: VAL**, keyboard_parts:HOLE_M3, F.Cu at (370.3, 207.1)
- added HOLE_M3: VAL**, keyboard_parts:HOLE_M3, F.Cu at (118.9, 206.6)
- added HOLE_M3: VAL**, keyboard_parts:HOLE_M3, F.Cu at (118.4, 126.5)
Other:
- board size 247.4 x 75.9 mm -> 259.4 x 87.9 mm
Changed lines of the file:
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@@
-(kicad_pcb (version 20171130) (host pcbnew "(5.1.5-0-10_14)")
+(kicad_pcb (version 20171130) (host pcbnew "(5.1.5)-3")
   (general
     (thickness 1.6)
@@
     (tracks 0)
     (zones 0)
-    (modules 47)
+    (modules 53)
     (nets 1)
   )
@@
     (mod_text_size 1 1)
     (mod_text_width 0.15)
-    (pad_size 2.5 3.08)
-    (pad_drill 1.5)
+    (pad_size 4 4)
+    (pad_drill 3.2)
     (pad_to_mask_clearance 0.051)
     (solder_mask_min_width 0.25)
@@
     (uvia_drill 0.1)
   )
+  (module keyboard_parts:HOLE_M3 (layer F.Cu)
+    (at 245.872 208.3985)
+    (fp_text reference HOLE_M3 (at 0 -4.5) (layer F.SilkS) hide
+      (effects (font (size 1.524 1.524) (thickness 0.3048)))
+    )
+    (fp_text value VAL** (at 0.05 -7.25) (layer F.SilkS) hide
+      (effects (font (size 1.524 1.524) (thickness 0.3048)))
+    )
+    (pad 1 thru_hole circle (at -1.55575 -1.778) (size 4 4) (drill 3.2) (layers *.Cu *.Mask F.SilkS))
+  )
+  (module keyboard_parts:HOLE_M3 (layer F.Cu)
+    (at 245.872 125.8485)
+    (fp_text reference HOLE_M3 (at 0 -4.5) (layer F.SilkS) hide
+      (effects (font (size 1.524 1.524) (thickness 0.3048)))
+    )
+    (fp_text value VAL** (at 0.05 -7.25) (layer F.SilkS) hide
+      (effects (font (size 1.524 1.524) (thickness 0.3048)))
+    )
+    (pad 1 thru_hole circle (at -1.55575 0.7155) (size 4 4) (drill 3.2) (layers *.Cu *.Mask F.SilkS))
+  )
+  (module keyboard_parts:HOLE_M3 (layer F.Cu)
+    (at 370.332 127.1185)
+    (fp_text reference HOLE_M3 (at 0 -4.5) (layer F.SilkS) hide
+      (effects (font (size 1.524 1.524) (thickness 0.3048)))
+    )
+    (fp_text value VAL** (at 0.05 -7.25) (layer F.SilkS) hide
+      (effects (font (size 1.524 1.524) (thickness 0.3048)))
+    )
+    (pad 1 thru_hole circle (at -0.2625 -0.5545) (size 4 4) (drill 3.2) (layers *.Cu *.Mask F.SilkS))
+  )
+  (module keyboard_parts:HOLE_M3 (layer F.Cu)
+    (at 370.332 207.1285)
+    (fp_text reference HOLE_M3 (at 0 -4.5) (layer F.SilkS) hide
+      (effects (font (size 1.524 1.524) (thickness 0.3048)))
+    )
+    (fp_text value VAL** (at 0.05 -7.25) (layer F.SilkS) hide
+      (effects (font (size 1.524 1.524) (thickness 0.3048)))
+    )
+    (pad 1 thru_hole circle (at -0.2625 -0.508) (size 4 4) (drill 3.2) (layers *.Cu *.Mask F.SilkS))
+  )
+  (module keyboard_parts:HOLE_M3 (layer F.Cu)
+    (at 118.872 206.6205)
+    (fp_text reference HOLE_M3 (at 0 -4.5) (layer F.SilkS) hide
+      (effects (font (size 1.524 1.524) (thickness 0.3048)))
+    )
+    (fp_text value VAL** (at 0.05 -7.25) (layer F.SilkS) hide
+      (effects (font (size 1.524 1.524) (thickness 0.3048)))
+    )
+    (pad 1 thru_hole circle (at -0.3725 0) (size 4 4) (drill 3.2) (layers *.Cu *.Mask F.SilkS))
+  )
+  (module keyboard_parts:HOLE_M3 (layer F.Cu)
+    (at 118.364 126.492)
+    (fp_text reference HOLE_M3 (at 0 -4.5) (layer F.SilkS) hide
+      (effects (font (size 1.524 1.524) (thickness 0.3048)))
+    )
+    (fp_text value VAL** (at 0.05 -7.25) (layer F.SilkS) hide
+      (effects (font (size 1.524 1.524) (thickness 0.3048)))
+    )
+    (pad 1 thru_hole circle (at 0.199 0.072) (size 4 4) (drill 3.2) (layers *.Cu *.Mask F.SilkS))
+  )
   (module keebs:Mx_Cutout_225 (layer B.Cu)
     (at 265.73125 195.15)
@@
     (fp_line (start -9.398 9.398) (end 9.398 9.398) (layer Dwgs.User) (width 0.1524))
   )
-  (gr_arc (start 122.9995 202.1205) (end 120.5865 202.1205) (angle -90) (layer Edge.Cuts) (width 0.05))
-  (gr_arc (start 365.5695 202.1205) (end 365.5695 204.5335) (angle -90) (layer Edge.Cuts) (width 0.05))
-  (gr_arc (start 365.5695 131.0005) (end 367.9825 131.0005) (angle -90) (layer Edge.Cuts) (width 0.05))
-  (gr_arc (start 123.063 131.064) (end 122.9995 128.5875) (angle -88.53119929) (layer Edge.Cuts) (width 0.05))
-  (gr_line (start 120.5865 202.1205) (end 120.5865 131.064) (layer Edge.Cuts) (width 0.05))
-  (gr_line (start 365.5695 204.5335) (end 122.9995 204.5335) (layer Edge.Cuts) (width 0.05))
-  (gr_line (start 367.9825 131.0005) (end 367.9825 202.1205) (layer Edge.Cuts) (width 0.05))
-  (gr_line (start 122.9995 128.5875) (end 365.5695 128.5875) (layer Edge.Cuts) (width 0.05))
+  (gr_arc (start 116.9995 208.1205) (end 114.5865 208.1205) (angle -90) (layer Edge.Cuts) (width 0.05))
+  (gr_arc (start 371.5695 208.1205) (end 371.5695 210.5335) (angle -90) (layer Edge.Cuts) (width 0.05))
+  (gr_arc (start 371.5695 125.0005) (end 373.9825 125.0005) (angle -90) (layer Edge.Cuts) (width 0.05))
+  (gr_arc (start 117.063 125.064) (end 116.9995 122.5875) (angle -88.53119929) (layer Edge.Cuts) (width 0.05))
+  (gr_line (start 114.5865 208.1205) (end 114.5865 125.064) (layer Edge.Cuts) (width 0.05))
+  (gr_line (start 371.5695 210.5335) (end 116.9995 210.5335) (layer Edge.Cuts) (width 0.05))
+  (gr_line (start 373.9825 125.0005) (end 373.9825 208.1205) (layer Edge.Cuts) (width 0.05))
+  (gr_line (start 116.9995 122.5875) (end 371.5695 122.5875) (layer Edge.Cuts) (width 0.05))
   (zone (net 0) (net_name "") (layer F.Cu) (hatch edge 0.508)
     (connect_pads (clearance 0.508))
@@
     (polygon
       (pts
-        (xy 380.111 218.948) (xy 109.982 215.265) (xy 112.776 125.603) (xy 116.205 125.73) (xy 377.825 123.19)
+        (xy 380.111 218.948) (xy 109.982 215.265) (xy 111.76 118.364) (xy 118.364 117.856) (xy 381 114.3)
       )
     )
@@
     (polygon
       (pts
-        (xy 384.81 219.837) (xy 108.077 215.646) (xy 110.744 122.555) (xy 378.587 122.174)
+        (xy 384.81 219.837) (xy 108.077 215.646) (xy 108.204 116.84) (xy 382.016 116.332)
       )
     )

Commit message: increased plate to 8mm extra
Parts:
- moved HOLE_M3 2.83 mm to (372.3, 125.1)
- moved HOLE_M3 2.83 mm to (372.3, 209.1)
- moved HOLE_M3 2.83 mm to (116.9, 208.6)
- moved HOLE_M3 2.83 mm to (116.4, 124.5)
- moved HOLE_M3 2.00 mm to (245.9, 210.4)
- moved HOLE_M3 2.00 mm to (245.9, 123.8)
Other:
- board size 259.4 x 87.9 mm -> 263.4 x 91.9 mm
Changed lines of the file:
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@@
   )
   (module keyboard_parts:HOLE_M3 (layer F.Cu)
-    (at 245.872 208.3985)
+    (at 245.872 210.3985)
     (fp_text reference HOLE_M3 (at 0 -4.5) (layer F.SilkS) hide
       (effects (font (size 1.524 1.524) (thickness 0.3048)))
@@
   )
   (module keyboard_parts:HOLE_M3 (layer F.Cu)
-    (at 245.872 125.8485)
+    (at 245.872 123.8485)
     (fp_text reference HOLE_M3 (at 0 -4.5) (layer F.SilkS) hide
       (effects (font (size 1.524 1.524) (thickness 0.3048)))
@@
   )
   (module keyboard_parts:HOLE_M3 (layer F.Cu)
-    (at 370.332 127.1185)
+    (at 372.332 125.1185)
     (fp_text reference HOLE_M3 (at 0 -4.5) (layer F.SilkS) hide
       (effects (font (size 1.524 1.524) (thickness 0.3048)))
@@
   )
   (module keyboard_parts:HOLE_M3 (layer F.Cu)
-    (at 370.332 207.1285)
+    (at 372.332 209.1285)
     (fp_text reference HOLE_M3 (at 0 -4.5) (layer F.SilkS) hide
       (effects (font (size 1.524 1.524) (thickness 0.3048)))
@@
   )
   (module keyboard_parts:HOLE_M3 (layer F.Cu)
-    (at 118.872 206.6205)
+    (at 116.872 208.6205)
     (fp_text reference HOLE_M3 (at 0 -4.5) (layer F.SilkS) hide
       (effects (font (size 1.524 1.524) (thickness 0.3048)))
@@
   )
   (module keyboard_parts:HOLE_M3 (layer F.Cu)
-    (at 118.364 126.492)
+    (at 116.364 124.492)
     (fp_text reference HOLE_M3 (at 0 -4.5) (layer F.SilkS) hide
       (effects (font (size 1.524 1.524) (thickness 0.3048)))
@@
     (fp_line (start -9.398 9.398) (end 9.398 9.398) (layer Dwgs.User) (width 0.1524))
   )
-  (gr_arc (start 116.9995 208.1205) (end 114.5865 208.1205) (angle -90) (layer Edge.Cuts) (width 0.05))
-  (gr_arc (start 371.5695 208.1205) (end 371.5695 210.5335) (angle -90) (layer Edge.Cuts) (width 0.05))
-  (gr_arc (start 371.5695 125.0005) (end 373.9825 125.0005) (angle -90) (layer Edge.Cuts) (width 0.05))
-  (gr_arc (start 117.063 125.064) (end 116.9995 122.5875) (angle -88.53119929) (layer Edge.Cuts) (width 0.05))
-  (gr_line (start 114.5865 208.1205) (end 114.5865 125.064) (layer Edge.Cuts) (width 0.05))
-  (gr_line (start 371.5695 210.5335) (end 116.9995 210.5335) (layer Edge.Cuts) (width 0.05))
-  (gr_line (start 373.9825 125.0005) (end 373.9825 208.1205) (layer Edge.Cuts) (width 0.05))
-  (gr_line (start 116.9995 122.5875) (end 371.5695 122.5875) (layer Edge.Cuts) (width 0.05))
+  (gr_arc (start 114.9995 210.1205) (end 112.5865 210.1205) (angle -90) (layer Edge.Cuts) (width 0.05))
+  (gr_arc (start 373.5695 210.1205) (end 373.5695 212.5335) (angle -90) (layer Edge.Cuts) (width 0.05))
+  (gr_arc (start 373.5695 123.0005) (end 375.9825 123.0005) (angle -90) (layer Edge.Cuts) (width 0.05))
+  (gr_arc (start 115.063 123.064) (end 114.9995 120.5875) (angle -88.53119929) (layer Edge.Cuts) (width 0.05))
+  (gr_line (start 112.5865 210.1205) (end 112.5865 123.064) (layer Edge.Cuts) (width 0.05))
+  (gr_line (start 373.5695 212.5335) (end 114.9995 212.5335) (layer Edge.Cuts) (width 0.05))
+  (gr_line (start 375.9825 123.0005) (end 375.9825 210.1205) (layer Edge.Cuts) (width 0.05))
+  (gr_line (start 114.9995 120.5875) (end 373.5695 120.5875) (layer Edge.Cuts) (width 0.05))
   (zone (net 0) (net_name "") (layer F.Cu) (hatch edge 0.508)
     (connect_pads (clearance 0.508))
