File: plate.kicad_pcb (KiCad board)
At the start: 2 copper layers, 263.4 x 91.9 mm, 53 parts, among them K101 KEYSW, K102 KEYSW, K103 KEYSW, K104 KEYSW, K105 KEYSW, K106 KEYSW, K107 KEYSW, K108 KEYSW, K109 KEYSW, K110 KEYSW, K111 KEYSW, K112 KEYSW, K113 KEYSW, K114 KEYSW, K115 KEYSW, K116 KEYSW, K118 KEYSW, K119 KEYSW, K120 KEYSW, K121 KEYSW, K122 KEYSW, K123 KEYSW, K124 KEYSW, K125 KEYSW, K126 KEYSW, K127 KEYSW, K128 KEYSW, K129 KEYSW, K130 KEYSW, K131 KEYSW, K132 KEYSW, K133 KEYSW, K134 KEYSW, K135 KEYSW, K136 KEYSW, K137 KEYSW, K138 KEYSW, K139 KEYSW, K140 KEYSW, K141 KEYSW, K142 KEYSW, K143 KEYSW, K144 KEYSW, K145 KEYSW, K146 KEYSW, K147 KEYSW, K148 KEYSW

Commit message: fixed soldering mask for 225, fixed placement of m3
Parts:
- moved HOLE_M3 1.78 mm to (245.9, 208.6)
- moved HOLE_M3 0.67 mm to (372.1, 124.5)
- moved HOLE_M3 0.65 mm to (245.9, 124.5)
- moved HOLE_M3 0.57 mm to (372.1, 208.6)
- moved HOLE_M3 0.31 mm to (116.6, 208.6)
- moved HOLE_M3 0.20 mm to (116.6, 124.5)
Changed lines of the file:
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@@
   )
   (module keyboard_parts:HOLE_M3 (layer F.Cu)
-    (at 245.872 210.3985)
+    (at 245.872 208.6205)
     (fp_text reference HOLE_M3 (at 0 -4.5) (layer F.SilkS) hide
       (effects (font (size 1.524 1.524) (thickness 0.3048)))
@@
   )
   (module keyboard_parts:HOLE_M3 (layer F.Cu)
-    (at 245.872 123.8485)
+    (at 245.872 124.5005)
     (fp_text reference HOLE_M3 (at 0 -4.5) (layer F.SilkS) hide
       (effects (font (size 1.524 1.524) (thickness 0.3048)))
@@
   )
   (module keyboard_parts:HOLE_M3 (layer F.Cu)
-    (at 372.332 125.1185)
+    (at 372.0695 124.5005)
     (fp_text reference HOLE_M3 (at 0 -4.5) (layer F.SilkS) hide
       (effects (font (size 1.524 1.524) (thickness 0.3048)))
@@
   )
   (module keyboard_parts:HOLE_M3 (layer F.Cu)
-    (at 372.332 209.1285)
+    (at 372.0695 208.6205)
     (fp_text reference HOLE_M3 (at 0 -4.5) (layer F.SilkS) hide
       (effects (font (size 1.524 1.524) (thickness 0.3048)))
@@
   )
   (module keyboard_parts:HOLE_M3 (layer F.Cu)
-    (at 116.872 208.6205)
+    (at 116.563 208.6205)
     (fp_text reference HOLE_M3 (at 0 -4.5) (layer F.SilkS) hide
       (effects (font (size 1.524 1.524) (thickness 0.3048)))
@@
   )
   (module keyboard_parts:HOLE_M3 (layer F.Cu)
-    (at 116.364 124.492)
+    (at 116.563 124.5005)
     (fp_text reference HOLE_M3 (at 0 -4.5) (layer F.SilkS) hide
       (effects (font (size 1.524 1.524) (thickness 0.3048)))
@@
       (effects (font (size 1.524 1.524) (thickness 0.3048)))
     )
-    (fp_poly (pts (xy 6.985 -6.985) (xy -6.985 -6.985) (xy -6.985 6.985) (xy 6.985 6.985)) (layer F.Mask) (width 2))
-    (fp_poly (pts (xy 6.985 -6.985) (xy -6.985 -6.985) (xy -6.985 6.985) (xy 6.985 6.985)) (layer B.Mask) (width 2))
+    (fp_poly (pts (xy -6.985 6.985) (xy 6.985 6.985) (xy 7.0104 5.4864) (xy 7.0104 5.6896)
+      (xy 8.6106 5.6896) (xy 15.2654 5.6896) (xy 15.2654 2.286) (xy 16.129 2.286)
+      (xy 16.129 -0.508) (xy 15.2654 -0.508) (xy 15.2654 -6.604) (xy 14.224 -6.604)
+      (xy 14.224 -7.7724) (xy 9.652 -7.7724) (xy 9.652 -6.604) (xy 9.7028 -5.842)
+      (xy 8.6106 -5.8166) (xy 6.985 -5.8166) (xy 6.985 -6.985) (xy -6.985 -6.985)
+      (xy -6.985 -5.8166) (xy -8.6106 -5.8166) (xy -9.652 -5.842) (xy -9.652 -6.604)
+      (xy -9.652 -7.7724) (xy -14.224 -7.7724) (xy -14.224 -6.604) (xy -15.2654 -6.604)
+      (xy -15.2654 -0.508) (xy -16.129 -0.508) (xy -16.129 2.286) (xy -15.2654 2.286)
+      (xy -15.2654 5.6896) (xy -8.6106 5.6896) (xy -6.0452 5.6896) (xy -6.985 4.8768)) (layer F.Mask) (width 2))
+    (fp_poly (pts (xy -6.985 6.985) (xy 6.985 6.985) (xy 7.0104 5.4864) (xy 7.0104 5.6896)
+      (xy 8.6106 5.6896) (xy 15.2654 5.6896) (xy 15.2654 2.286) (xy 16.129 2.286)
+      (xy 16.129 -0.508) (xy 15.2654 -0.508) (xy 15.2654 -6.604) (xy 14.224 -6.604)
+      (xy 14.224 -7.7724) (xy 9.652 -7.7724) (xy 9.652 -6.604) (xy 9.7028 -5.842)
+      (xy 8.6106 -5.8166) (xy 6.985 -5.8166) (xy 6.985 -6.985) (xy -6.985 -6.985)
+      (xy -6.985 -5.8166) (xy -8.6106 -5.8166) (xy -9.652 -5.842) (xy -9.652 -6.604)
+      (xy -9.652 -7.7724) (xy -14.224 -7.7724) (xy -14.224 -6.604) (xy -15.2654 -6.604)
+      (xy -15.2654 -0.508) (xy -16.129 -0.508) (xy -16.129 2.286) (xy -15.2654 2.286)
+      (xy -15.2654 5.6896) (xy -8.6106 5.6896) (xy -6.0452 5.6896) (xy -6.985 4.8768)) (layer B.Mask) (width 2))
     (fp_line (start -6.985 4.8768) (end -6.985 6.985) (layer Eco2.User) (width 0.1524))
     (fp_line (start -8.6106 4.8768) (end -6.985 4.8768) (layer Eco2.User) (width 0.1524))
@@
       (effects (font (size 1.524 1.524) (thickness 0.3048)))
     )
-    (fp_poly (pts (xy 6.985 -6.985) (xy -6.985 -6.985) (xy -6.985 6.985) (xy 6.985 6.985)) (layer F.Mask) (width 2))
-    (fp_poly (pts (xy 6.985 -6.985) (xy -6.985 -6.985) (xy -6.985 6.985) (xy 6.985 6.985)) (layer B.Mask) (width 2))
+    (fp_poly (pts (xy -6.985 6.985) (xy 6.985 6.985) (xy 7.0104 5.4864) (xy 7.0104 5.6896)
+      (xy 8.6106 5.6896) (xy 15.2654 5.6896) (xy 15.2654 2.286) (xy 16.129 2.286)
+      (xy 16.129 -0.508) (xy 15.2654 -0.508) (xy 15.2654 -6.604) (xy 14.224 -6.604)
+      (xy 14.224 -7.7724) (xy 9.652 -7.7724) (xy 9.652 -6.604) (xy 9.7028 -5.842)
+      (xy 8.6106 -5.8166) (xy 6.985 -5.8166) (xy 6.985 -6.985) (xy -6.985 -6.985)
+      (xy -6.985 -5.8166) (xy -8.6106 -5.8166) (xy -9.652 -5.842) (xy -9.652 -6.604)
+      (xy -9.652 -7.7724) (xy -14.224 -7.7724) (xy -14.224 -6.604) (xy -15.2654 -6.604)
+      (xy -15.2654 -0.508) (xy -16.129 -0.508) (xy -16.129 2.286) (xy -15.2654 2.286)
+      (xy -15.2654 5.6896) (xy -8.6106 5.6896) (xy -6.0452 5.6896) (xy -6.985 4.8768)) (layer F.Mask) (width 2))
+    (fp_poly (pts (xy -6.985 6.985) (xy 6.985 6.985) (xy 7.0104 5.4864) (xy 7.0104 5.6896)
+      (xy 8.6106 5.6896) (xy 15.2654 5.6896) (xy 15.2654 2.286) (xy 16.129 2.286)
+      (xy 16.129 -0.508) (xy 15.2654 -0.508) (xy 15.2654 -6.604) (xy 14.224 -6.604)
+      (xy 14.224 -7.7724) (xy 9.652 -7.7724) (xy 9.652 -6.604) (xy 9.7028 -5.842)
+      (xy 8.6106 -5.8166) (xy 6.985 -5.8166) (xy 6.985 -6.985) (xy -6.985 -6.985)
+      (xy -6.985 -5.8166) (xy -8.6106 -5.8166) (xy -9.652 -5.842) (xy -9.652 -6.604)
+      (xy -9.652 -7.7724) (xy -14.224 -7.7724) (xy -14.224 -6.604) (xy -15.2654 -6.604)
+      (xy -15.2654 -0.508) (xy -16.129 -0.508) (xy -16.129 2.286) (xy -15.2654 2.286)
+      (xy -15.2654 5.6896) (xy -8.6106 5.6896) (xy -6.0452 5.6896) (xy -6.985 4.8768)) (layer B.Mask) (width 2))
     (fp_line (start -6.985 4.8768) (end -6.985 6.985) (layer Eco2.User) (width 0.1524))
     (fp_line (start -8.6106 4.8768) (end -6.985 4.8768) (layer Eco2.User) (width 0.1524))
